Commit message: Update robotiq_arg2f_140_model_macro.xacro

File: src/robotiq_arg85_description/urdf/robotiq_arg2f_140_model_macro.xacro (robot description, xacro)
@@ -145,5 +145,5 @@
       <child link="${prefix}${fingerprefix}_inner_finger" />
       <axis xyz="1 0 0" />
-      <limit lower="0" upper="0.8757" velocity="2.0" effort="1000" />
+      <limit lower="-0.1" upper="0.8757" velocity="2.0" effort="1000" />
       <!--  <mimic joint="${prefix}finger_joint" multiplier="1" offset="0" /> -->
     </joint>
