Commit message: Update maci.urdf.xacro

File: src/maci/robot_description/maci.urdf.xacro (robot description, xacro)
@@ -17,5 +17,5 @@
     <!-- Lets add a realsense camera to give some depth perception to Maci. -->
     <xacro:realsense world_link_name="world">
-        <origin xyz="0 1.00 1.2" rpy="0 ${pi/4} -${pi/2}" />
+        <origin xyz="0 2.00 2.2" rpy="0 ${pi/4} -${pi/2}" />
     </xacro:realsense>
     <xacro:macro name="ros2_position_controller" params="joint_name">

Commit message: Update maci.urdf.xacro

File: src/maci/robot_description/maci.urdf.xacro (robot description, xacro)
@@ -16,6 +16,6 @@
     </joint>
     <!-- Lets add a realsense camera to give some depth perception to Maci. -->
-    <xacro:realsense world_link_name="world">
-        <origin xyz="0 2.00 2.2" rpy="0 ${pi/4} -${pi/2}" />
+    <xacro:realsense world_link_name="ur5_base_link">
+        <origin xyz="0 -2.00 -2.2" rpy="0 -${pi/4} ${pi/2}" />
     </xacro:realsense>
     <xacro:macro name="ros2_position_controller" params="joint_name">
